File: hw/Synthetic-Fireflies.kicad_sch (KiCad schematic)
At the start: 0 parts

Commit message: Complete MCU Power section of HW design guide
Other:
- added sheet MCU (MCU.kicad_sch)
- added sheet Power (Power.kicad_sch)
Changed lines of the file:
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@@
-(kicad_sch (version 20211123) (generator eeschema)
+(kicad_sch (version 20230121) (generator eeschema)
   (paper "A3")
   (title_block
     (title "Top Level")
   )
+  (sheet (at 25.4 129.54) (size 41.91 24.13) (fields_autoplaced)
+    (stroke (width 0.1524) (type solid))
+    (fill (color 0 0 0 0.0000))
+    (property "Sheetname" "Power" (at 25.4 128.8284 0)
+      (effects (font (size 1.27 1.27)) (justify left bottom))
+    )
+    (property "Sheetfile" "Power.kicad_sch" (at 25.4 154.2546 0)
+      (effects (font (size 1.27 1.27)) (justify left top))
+    )
+    (instances
+      (project "Synthetic-Fireflies"
+        (path "/eb7890aa-4169-47c5-87d4-a9440f7befdd" (page "2"))
+      )
+    )
+  )
+  (sheet (at 101.6 129.54) (size 41.91 24.13) (fields_autoplaced)
+    (stroke (width 0.1524) (type solid))
+    (fill (color 0 0 0 0.0000))
+    (property "Sheetname" "MCU" (at 101.6 128.8284 0)
+      (effects (font (size 1.27 1.27)) (justify left bottom))
+    )
+    (property "Sheetfile" "MCU.kicad_sch" (at 101.6 154.2546 0)
+      (effects (font (size 1.27 1.27)) (justify left top))
+    )
+    (instances
+      (project "Synthetic-Fireflies"
+        (path "/eb7890aa-4169-47c5-87d4-a9440f7befdd" (page "3"))
+      )
+    )
+  )
   (sheet_instances
